Commit message: Completed the macro for the second part of the assignment

File: urdf/joint_model.urdf (robot description, URDF)
Before this commit: robot qube_model, 5 links, 4 joints
Links:
- removed link angle_link
- removed link base_link
- removed link rotor_link
- removed link stator_link
- removed link world
Joints:
- removed joint angle
- removed joint base_joint
- removed joint indicator
- removed joint stator_joint
